File: KiCAD/ALU.kicad_sch (KiCad schematic)
At the start: 27 parts, among them J17 ALU_A, J18 ALU_B, J19 ALU_OUT, J20 ALU_FLGS, U5 74HCT86, U51 74HCT21, U57 74HCT04, U64 74HCT74, U66 74HCT574, U67 74HCT574, U68 74HCT574, U69 74LS181, U70 74LS181, U71 74HCT27, U72 74HCT02, U73 74HCT541

Commit message: Cleanup of KiCad files and adding board PDFs
Parts:
- C101, C102, C105, C107: footprint Project Library:C_Disc_D7.5mm_W2.5mm_P7.62mm -> Project Library:C_Disc_D7.5mm_W2.5mm_P7.62mm_pol
Changed lines of the file:
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@@
 			)
 		)
-		(property "Footprint" "Project Library:C_Disc_D7.5mm_W2.5mm_P7.62mm"
+		(property "Footprint" "Project Library:C_Disc_D7.5mm_W2.5mm_P7.62mm_pol"
 			(at 158.75 48.26 0)
 			(effects
@@
 			)
 		)
-		(property "Footprint" "Project Library:C_Disc_D7.5mm_W2.5mm_P7.62mm"
+		(property "Footprint" "Project Library:C_Disc_D7.5mm_W2.5mm_P7.62mm_pol"
 			(at 67.31 152.4 0)
 			(effects
@@
 			)
 		)
-		(property "Footprint" "Project Library:C_Disc_D7.5mm_W2.5mm_P7.62mm"
+		(property "Footprint" "Project Library:C_Disc_D7.5mm_W2.5mm_P7.62mm_pol"
 			(at 232.41 80.01 0)
 			(effects
@@
 			)
 		)
-		(property "Footprint" "Project Library:C_Disc_D7.5mm_W2.5mm_P7.62mm"
+		(property "Footprint" "Project Library:C_Disc_D7.5mm_W2.5mm_P7.62mm_pol"
 			(at 67.31 35.56 0)
 			(effects
