File: KiCAD/Clock_and_Reset.kicad_sch (KiCad schematic)
At the start: 46 parts, among them SW1 STEP, SW2 RESET, SW3 SW_Rotary_SS-10-16, U1 74HCT04, U10 74HCT11, U11 74HCT74, U12 74HCT74, U2 LM555, U3 74HCT14, U4 74HCT74, U5 74HCT86, U6 74HCT02, U7 74HCT73, U8 74HCT73, U9 74HCT74, Y1 4MHz/30pF

Commit message: Cleanup of KiCad files and adding board PDFs
Parts:
- C10, C6, C7, C8, C9: footprint Project Library:C_Disc_D7.5mm_W2.5mm_P7.62mm -> Project Library:C_Disc_D7.5mm_W2.5mm_P7.62mm_pol
Changed lines of the file:
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@@
 			)
 		)
-		(property "Footprint" "Project Library:C_Disc_D7.5mm_W2.5mm_P7.62mm"
+		(property "Footprint" "Project Library:C_Disc_D7.5mm_W2.5mm_P7.62mm_pol"
 			(at 124.46 195.58 0)
 			(effects
@@
 			)
 		)
-		(property "Footprint" "Project Library:C_Disc_D7.5mm_W2.5mm_P7.62mm"
+		(property "Footprint" "Project Library:C_Disc_D7.5mm_W2.5mm_P7.62mm_pol"
 			(at 132.08 195.58 0)
 			(effects
@@
 			)
 		)
-		(property "Footprint" "Project Library:C_Disc_D7.5mm_W2.5mm_P7.62mm"
+		(property "Footprint" "Project Library:C_Disc_D7.5mm_W2.5mm_P7.62mm_pol"
 			(at 53.34 124.46 0)
 			(effects
@@
 			)
 		)
-		(property "Footprint" "Project Library:C_Disc_D7.5mm_W2.5mm_P7.62mm"
+		(property "Footprint" "Project Library:C_Disc_D7.5mm_W2.5mm_P7.62mm_pol"
 			(at 147.32 195.58 0)
 			(effects
@@
 			)
 		)
-		(property "Footprint" "Project Library:C_Disc_D7.5mm_W2.5mm_P7.62mm"
+		(property "Footprint" "Project Library:C_Disc_D7.5mm_W2.5mm_P7.62mm_pol"
 			(at 139.7 195.58 0)
 			(effects
