File: KiCAD/Exception_Handling.kicad_sch (KiCad schematic)
At the start: 27 parts, among them U45 74HCT11, U57 74HCT04, U58 74HCT08, U59 74HCT74, U6 74HCT02, U60 74HCT32, U61 74HCT27, U62 74HCT173, U63 74HCT74, U64 74HCT74, U65 74HCT574, U7 74HCT73

Commit message: Cleanup of KiCad files and adding board PDFs
Parts:
- C87, C90, C93: footprint Project Library:C_Disc_D7.5mm_W2.5mm_P7.62mm -> Project Library:C_Disc_D7.5mm_W2.5mm_P7.62mm_pol
Changed lines of the file:
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@@
 			)
 		)
-		(property "Footprint" "Project Library:C_Disc_D7.5mm_W2.5mm_P7.62mm"
+		(property "Footprint" "Project Library:C_Disc_D7.5mm_W2.5mm_P7.62mm_pol"
 			(at 92.71 144.78 0)
 			(effects
@@
 			)
 		)
-		(property "Footprint" "Project Library:C_Disc_D7.5mm_W2.5mm_P7.62mm"
+		(property "Footprint" "Project Library:C_Disc_D7.5mm_W2.5mm_P7.62mm_pol"
 			(at 181.61 58.42 0)
 			(effects
@@
 			)
 		)
-		(property "Footprint" "Project Library:C_Disc_D7.5mm_W2.5mm_P7.62mm"
+		(property "Footprint" "Project Library:C_Disc_D7.5mm_W2.5mm_P7.62mm_pol"
 			(at 217.17 149.86 0)
 			(effects
