File: KiCAD/External_Memory.kicad_sch (KiCad schematic)
At the start: 19 parts, among them J23 ABL, J24 ABH, J25 DB, U102 HM62256BLP, U103 GAL16V8, U104 HM62256BLP, U105 SST39SF010, U57 74HCT04, U97 74HCT139

Commit message: Cleanup of KiCad files and adding board PDFs
Parts:
- C154, C155, C157, C159: footprint Project Library:C_Disc_D7.5mm_W2.5mm_P7.62mm -> Project Library:C_Disc_D7.5mm_W2.5mm_P7.62mm_pol
Changed lines of the file:
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@@
 			)
 		)
-		(property "Footprint" "Project Library:C_Disc_D7.5mm_W2.5mm_P7.62mm"
+		(property "Footprint" "Project Library:C_Disc_D7.5mm_W2.5mm_P7.62mm_pol"
 			(at 146.05 29.21 0)
 			(effects
@@
 			)
 		)
-		(property "Footprint" "Project Library:C_Disc_D7.5mm_W2.5mm_P7.62mm"
+		(property "Footprint" "Project Library:C_Disc_D7.5mm_W2.5mm_P7.62mm_pol"
 			(at 83.82 119.38 0)
 			(effects
@@
 			)
 		)
-		(property "Footprint" "Project Library:C_Disc_D7.5mm_W2.5mm_P7.62mm"
+		(property "Footprint" "Project Library:C_Disc_D7.5mm_W2.5mm_P7.62mm_pol"
 			(at 82.55 29.21 0)
 			(effects
@@
 			)
 		)
-		(property "Footprint" "Project Library:C_Disc_D7.5mm_W2.5mm_P7.62mm"
+		(property "Footprint" "Project Library:C_Disc_D7.5mm_W2.5mm_P7.62mm_pol"
 			(at 205.74 29.21 0)
 			(effects
