File: KiCAD/Instruction_Decoder.kicad_sch (KiCad schematic)
At the start: 35 parts, among them U30 74HCT32, U44 74HCT21, U45 74HCT11, U46 74HCT138, U47 74HCT138, U48 74HCT138, U49 74HCT08, U50 74HCT08, U51 74HCT21, U52 74HCT08, U53 74HCT00, U54 74HCT138, U55 74HCT138, U56 74HCT138, U57 74HCT04, U58 74HCT08

Commit message: Cleanup of KiCad files and adding board PDFs
Parts:
- C82, C83, C84, C85: footprint Project Library:C_Disc_D7.5mm_W2.5mm_P7.62mm -> Project Library:C_Disc_D7.5mm_W2.5mm_P7.62mm_pol
Changed lines of the file:
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@@
 			)
 		)
-		(property "Footprint" "Project Library:C_Disc_D7.5mm_W2.5mm_P7.62mm"
+		(property "Footprint" "Project Library:C_Disc_D7.5mm_W2.5mm_P7.62mm_pol"
 			(at 238.76 175.26 0)
 			(effects
@@
 			)
 		)
-		(property "Footprint" "Project Library:C_Disc_D7.5mm_W2.5mm_P7.62mm"
+		(property "Footprint" "Project Library:C_Disc_D7.5mm_W2.5mm_P7.62mm_pol"
 			(at 254 175.26 0)
 			(effects
@@
 			)
 		)
-		(property "Footprint" "Project Library:C_Disc_D7.5mm_W2.5mm_P7.62mm"
+		(property "Footprint" "Project Library:C_Disc_D7.5mm_W2.5mm_P7.62mm_pol"
 			(at 261.62 175.26 0)
 			(effects
@@
 			)
 		)
-		(property "Footprint" "Project Library:C_Disc_D7.5mm_W2.5mm_P7.62mm"
+		(property "Footprint" "Project Library:C_Disc_D7.5mm_W2.5mm_P7.62mm_pol"
 			(at 246.38 175.26 0)
 			(effects
