File: KiCAD/Miscellaneous.kicad_sch (KiCad schematic)
At the start: 21 parts, among them J26 USB_C_Power, J27 Expansion, J28 UART, U1 74HCT04, U106 MC6850, U3 74HCT14, U52 74HCT08, U58 74HCT08, U60 74HCT32, U72 74HCT02, U83 74HCT86, U86 74HCT10, U9 74HCT74, Y2 1.8432MHz/30pF

Commit message: Cleanup of KiCad files and adding board PDFs
Parts:
- C163: footprint Project Library:C_Disc_D7.5mm_W2.5mm_P7.62mm -> Project Library:C_Disc_D7.5mm_W2.5mm_P7.62mm_pol
Changed lines of the file:
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@@
 	)
 	(junction
-		(at 135.89 172.72)
-		(diameter 0)
-		(color 0 0 0 0)
-	)
-	(junction
 		(at 86.36 31.75)
 		(diameter 0)
@@
 	)
 	(junction
-		(at 135.89 170.18)
-		(diameter 0)
-		(color 0 0 0 0)
-	)
-	(junction
 		(at 144.78 77.47)
 		(diameter 0)
@@
 	(wire
 		(pts
-			(xy 137.16 167.64) (xy 135.89 167.64)
-		)
-		(stroke
-			(width 0)
-			(type default)
-		)
-	)
-	(wire
-		(pts
 			(xy 83.82 59.69) (xy 87.63 59.69)
 		)
@@
 	(wire
 		(pts
-			(xy 135.89 172.72) (xy 135.89 175.26)
-		)
-		(stroke
-			(width 0)
-			(type default)
-		)
-	)
-	(wire
-		(pts
 			(xy 196.85 85.09) (xy 196.85 87.63)
 		)
@@
 	(wire
 		(pts
-			(xy 135.89 167.64) (xy 135.89 170.18)
-		)
-		(stroke
-			(width 0)
-			(type default)
-		)
-	)
-	(wire
-		(pts
 			(xy 86.36 31.75) (xy 87.63 31.75)
 		)
@@
 	(wire
 		(pts
-			(xy 135.89 172.72) (xy 137.16 172.72)
-		)
-		(stroke
-			(width 0)
-			(type default)
-		)
-	)
-	(wire
-		(pts
 			(xy 58.42 167.64) (xy 58.42 170.18)
 		)
@@
 	(wire
 		(pts
-			(xy 135.89 170.18) (xy 137.16 170.18)
-		)
-		(stroke
-			(width 0)
-			(type default)
-		)
-	)
-	(wire
-		(pts
 			(xy 27.94 151.13) (xy 27.94 148.59)
 		)
@@
 	(wire
 		(pts
-			(xy 135.89 170.18) (xy 135.89 172.72)
-		)
-		(stroke
-			(width 0)
-			(type default)
-		)
-	)
-	(wire
-		(pts
 			(xy 232.41 95.25) (xy 233.68 95.25)
 		)
@@
 	)
 	(symbol
-		(lib_id "power:GND")
-		(at 135.89 175.26 0)
-		(unit 1)
-		(exclude_from_sim no)
-		(in_bom yes)
-		(on_board yes)
-		(dnp no)
-		(fields_autoplaced yes)
-		(property "Reference" "#PWR0493"
-			(at 135.89 181.61 0)
-			(effects
-				(font
-					(size 1.27 1.27)
-				)
-				(hide yes)
-			)
-		)
-		(property "Value" "GND"
-			(at 135.89 180.34 0)
-			(effects
-				(font
-					(size 1.27 1.27)
-				)
-				(hide yes)
-			)
-		)
-		(property "Footprint" ""
-			(at 135.89 175.26 0)
-			(effects
-				(font
-					(size 1.27 1.27)
-				)
-				(hide yes)
-			)
-		)
-		(property "Datasheet" ""
-			(at 135.89 175.26 0)
-			(effects
-				(font
-					(size 1.27 1.27)
-				)
-				(hide yes)
-			)
-		)
-		(property "Description" "Power symbol creates a global label with name \"GND\" , ground"
-			(at 135.89 175.26 0)
-			(effects
-				(font
-					(size 1.27 1.27)
-				)
-				(hide yes)
-			)
-		)
-		(pin "1"
-		)
-		(instances
-			(project "TTL 6510 Computer"
-				(path "/a212c6c5-fafd-4da9-bbe3-09155431f13a/93b7d6b4-51bf-42e3-8ce0-2b824dfac93f"
-					(reference "#PWR0493")
-					(unit 1)
-				)
-			)
-		)
-	)
-	(symbol
 		(lib_id "Connector:Conn_01x06_Pin")
 		(at 238.76 100.33 0)
@@
 			)
 		)
-		(property "Footprint" "Project Library:C_Disc_D7.5mm_W2.5mm_P7.62mm"
+		(property "Footprint" "Project Library:C_Disc_D7.5mm_W2.5mm_P7.62mm_pol"
 			(at 218.44 22.86 0)
 			(effects
