File: KiCAD/Program_Counter.kicad_sch (KiCad schematic)
At the start: 24 parts, among them J1 PCL, J2 PCH, U13 74HCT541, U14 74HCT161, U15 74HCT541, U16 74HCT161, U17 74HCT541, U18 74HCT161, U19 74HCT541, U20 74HCT161, U6 74HCT02

Commit message: Cleanup of KiCad files and adding board PDFs
Parts:
- C26, C29, C30, C31: footprint Project Library:C_Disc_D7.5mm_W2.5mm_P7.62mm -> Project Library:C_Disc_D7.5mm_W2.5mm_P7.62mm_pol
Changed lines of the file:
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@@
 			)
 		)
-		(property "Footprint" "Project Library:C_Disc_D7.5mm_W2.5mm_P7.62mm"
+		(property "Footprint" "Project Library:C_Disc_D7.5mm_W2.5mm_P7.62mm_pol"
 			(at 199.39 173.99 0)
 			(effects
@@
 			)
 		)
-		(property "Footprint" "Project Library:C_Disc_D7.5mm_W2.5mm_P7.62mm"
+		(property "Footprint" "Project Library:C_Disc_D7.5mm_W2.5mm_P7.62mm_pol"
 			(at 173.99 173.99 0)
 			(effects
@@
 			)
 		)
-		(property "Footprint" "Project Library:C_Disc_D7.5mm_W2.5mm_P7.62mm"
+		(property "Footprint" "Project Library:C_Disc_D7.5mm_W2.5mm_P7.62mm_pol"
 			(at 186.69 173.99 0)
 			(effects
@@
 			)
 		)
-		(property "Footprint" "Project Library:C_Disc_D7.5mm_W2.5mm_P7.62mm"
+		(property "Footprint" "Project Library:C_Disc_D7.5mm_W2.5mm_P7.62mm_pol"
 			(at 212.09 173.99 0)
 			(effects
