File: KiCAD/Registers_and_DB_Driver.kicad_sch (KiCad schematic)
At the start: 14 parts, among them J10 Y, J8 A, J9 X, U21 74HCT08, U34 74HCT574, U35 74HCT245, U36 74HCT574, U37 74HCT574

Commit message: Cleanup of KiCad files and adding board PDFs
Parts:
- C56, C58: footprint Project Library:C_Disc_D7.5mm_W2.5mm_P7.62mm -> Project Library:C_Disc_D7.5mm_W2.5mm_P7.62mm_pol
Changed lines of the file:
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@@
 			)
 		)
-		(property "Footprint" "Project Library:C_Disc_D7.5mm_W2.5mm_P7.62mm"
+		(property "Footprint" "Project Library:C_Disc_D7.5mm_W2.5mm_P7.62mm_pol"
 			(at 200.66 162.56 0)
 			(effects
@@
 			)
 		)
-		(property "Footprint" "Project Library:C_Disc_D7.5mm_W2.5mm_P7.62mm"
+		(property "Footprint" "Project Library:C_Disc_D7.5mm_W2.5mm_P7.62mm_pol"
 			(at 187.96 162.56 0)
 			(effects
