File: KiCAD/Special_Conditions.kicad_sch (KiCad schematic)
At the start: 32 parts, among them U53 74HCT00, U59 74HCT74, U60 74HCT32, U76 74HCT32, U82 74HCT08, U83 74HCT86, U84 74HCT74, U85 74HCT00, U86 74HCT10, U87 74HCT125, U88 74HCT32, U89 74HCT74, U90 74HCT74, U91 74HCT74, U92 74HCT151

Commit message: Cleanup of KiCad files and adding board PDFs
Parts:
- C123, C124, C125, C127: footprint Project Library:C_Disc_D7.5mm_W2.5mm_P7.62mm -> Project Library:C_Disc_D7.5mm_W2.5mm_P7.62mm_pol
Changed lines of the file:
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@@
 			)
 		)
-		(property "Footprint" "Project Library:C_Disc_D7.5mm_W2.5mm_P7.62mm"
+		(property "Footprint" "Project Library:C_Disc_D7.5mm_W2.5mm_P7.62mm_pol"
 			(at 133.35 195.58 0)
 			(effects
@@
 			)
 		)
-		(property "Footprint" "Project Library:C_Disc_D7.5mm_W2.5mm_P7.62mm"
+		(property "Footprint" "Project Library:C_Disc_D7.5mm_W2.5mm_P7.62mm_pol"
 			(at 152.4 195.58 0)
 			(effects
@@
 			)
 		)
-		(property "Footprint" "Project Library:C_Disc_D7.5mm_W2.5mm_P7.62mm"
+		(property "Footprint" "Project Library:C_Disc_D7.5mm_W2.5mm_P7.62mm_pol"
 			(at 139.7 195.58 0)
 			(effects
@@
 			)
 		)
-		(property "Footprint" "Project Library:C_Disc_D7.5mm_W2.5mm_P7.62mm"
+		(property "Footprint" "Project Library:C_Disc_D7.5mm_W2.5mm_P7.62mm_pol"
 			(at 146.05 195.58 0)
 			(effects
