File: KiCAD/Status_Register.kicad_sch (KiCad schematic)
At the start: 28 parts, among them J21 SR, U45 74HCT11, U51 74HCT21, U52 74HCT08, U71 74HCT27, U72 74HCT02, U74 74HCT153, U75 74HCT153, U76 74HCT32, U77 74HCT74, U78 74HCT74, U79 74HCT74, U80 74HCT138, U81 74HCT541

Commit message: Cleanup of KiCad files and adding board PDFs
Parts:
- C110, C114, C115, C117: footprint Project Library:C_Disc_D7.5mm_W2.5mm_P7.62mm -> Project Library:C_Disc_D7.5mm_W2.5mm_P7.62mm_pol
Changed lines of the file:
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@@
 			)
 		)
-		(property "Footprint" "Project Library:C_Disc_D7.5mm_W2.5mm_P7.62mm"
+		(property "Footprint" "Project Library:C_Disc_D7.5mm_W2.5mm_P7.62mm_pol"
 			(at 224.79 132.08 0)
 			(effects
@@
 			)
 		)
-		(property "Footprint" "Project Library:C_Disc_D7.5mm_W2.5mm_P7.62mm"
+		(property "Footprint" "Project Library:C_Disc_D7.5mm_W2.5mm_P7.62mm_pol"
 			(at 209.55 132.08 0)
 			(effects
@@
 			)
 		)
-		(property "Footprint" "Project Library:C_Disc_D7.5mm_W2.5mm_P7.62mm"
+		(property "Footprint" "Project Library:C_Disc_D7.5mm_W2.5mm_P7.62mm_pol"
 			(at 201.93 132.08 0)
 			(effects
@@
 			)
 		)
-		(property "Footprint" "Project Library:C_Disc_D7.5mm_W2.5mm_P7.62mm"
+		(property "Footprint" "Project Library:C_Disc_D7.5mm_W2.5mm_P7.62mm_pol"
 			(at 217.17 132.08 0)
 			(effects
